File: hw/tft-lcd.sch (KiCad schematic (older format))
At the start: 10 parts, among them J301 HEADER_MOLEX_54104-4031, U301 FT812, U302 LED_DRIVER_MIC2289

Commit message: 1.7.0 pcb created, not yet ordered
Parts:
- removed C305: 100nF, kemet:0603, symbol 100nF
- removed C306: T491D226K035AT, kemet:7343, symbol T491D226K035AT
- removed R302: R_2OHM, usevolt:0603, symbol R_2OHM
- removed U302: LED_DRIVER_MIC2289, usevolt:MLF_8, symbol LED_DRIVER_MIC2289
- added C303: 100nF, kemet:0603, symbol 100nF
- added C304: CAP_EEE-FK1H470P, usevolt:CAP_EEE-FK1H470P, symbol CAP_EEE-FK1H470P
- added D301: DIODE_RS07J-GS18, usevolt:DO219AB, symbol DIODE_RS07J-GS18
- added J302: HEADER_MOLEX_52207-0433, usevolt:HEADER_MOLEX_52207-0433, symbol HEADER_MOLEX_52207-0433
- added R302: R_0.33OHM, usevolt:0603, symbol R_0.33OHM
- added U302: AL8805W5-7_LED_DRIVER, usevolt:SOT-25, symbol AL8805W5-7_LED_DRIVER
Connections:
- net labels added: VEE
- net labels removed: +5V
- wire segments 85 -> 88
