File: hw/tft-lcd.sch (KiCad schematic (older format))
At the start: 12 parts, among them J301 HEADER_MOLEX_54104-4031, J302 HEADER_MOLEX_52207-0433, U301 FT812, U302 AL8805W5-7_LED_DRIVER

Commit message: kicad schematic update
Parts:
- C301, C302, C303: symbol 100nF -> kemet:100nF
- C304: symbol CAP_EEE-FK1H470P -> usevolt:CAP_EEE-FK1H470P
- D301: symbol DIODE_RS07J-GS18 -> usevolt:DIODE_RS07J-GS18
- J301: symbol HEADER_MOLEX_54104-4031 -> usevolt:HEADER_MOLEX_54104-4031
- J302: symbol HEADER_MOLEX_52207-0433 -> usevolt:HEADER_MOLEX_52207-0433
- L301: symbol IND_744045210 -> usevolt:IND_744045210
- R301: symbol 10K -> multicomp:10K
- R302: symbol R_0.33OHM -> usevolt:R_0.33OHM
- U301: symbol FT812 -> usevolt:FT812
- U302: symbol AL8805W5-7_LED_DRIVER -> usevolt:AL8805W5-7_LED_DRIVER
Connections:
- wire segments 88 -> 105
Changed lines of the file:
@@
-EESchema Schematic File Version 2
-LIBS:display-rescue
-LIBS:kemet
-LIBS:multicomp
-LIBS:usevolt
-LIBS:wurth_elektronik_LED
-LIBS:power
+EESchema Schematic File Version 4
 LIBS:display-cache
 EELAYER 26 0
@@
 $EndDescr
 $Comp
-L HEADER_MOLEX_54104-4031 J301
+L usevolt:HEADER_MOLEX_54104-4031 J301
 U 1 1 58FC4B22
 P 9550 3250
@@
 YU
 $Comp
-L GND #PWR308
+L power1:GND #PWR308
 U 1 1 58FC5C8D
 P 8900 5800
@@
 $EndComp
 Wire Wire Line
-	8900 2000 8900 5800
+	8900 2000 8900 4600
 Connection ~ 8900 5300
 Connection ~ 8900 4600
@@
 	8800 1500 8800 2100
 $Comp
-L +3V3 #PWR303
+L power1:+3V3 #PWR303
 U 1 1 58FC70E1
 P 2650 2100
@@
 $EndComp
 Wire Wire Line
-	2650 2100 2650 2500
-Wire Wire Line
-	1300 2200 2850 2200
+	2650 2100 2650 2200
+Wire Wire Line
+	1300 2200 1650 2200
 Wire Wire Line
 	2650 2300 2850 2300
@@
 	2450 3200 2850 3200
 $Comp
-L GND #PWR304
+L power1:GND #PWR304
 U 1 1 58FC8063
 P 2650 5800
@@
 $EndComp
 Wire Wire Line
-	2650 5300 2650 5800
+	2650 5300 2650 5400
 Wire Wire Line
 	2650 5700 2850 5700
@@
 Connection ~ 2650 5400
 $Comp
-L 100nF C302
+L kemet:100nF C302
 U 1 1 58FC823D
 P 1650 2300
@@
 $EndComp
 $Comp
-L 100nF C301
+L kemet:100nF C301
 U 1 1 58FC82A4
 P 1300 2300
@@
 Connection ~ 1650 2200
 $Comp
-L GND #PWR301
+L power1:GND #PWR301
 U 1 1 58FC846A
 P 1300 2550
@@
 	1300 2550 1300 2500
 $Comp
-L +3V3 #PWR302
+L power1:+3V3 #PWR302
 U 1 1 5900C7EB
 P 1400 3150
@@
 	8450 1800 9400 1800
 $Comp
-L +3V3 #PWR307
+L power1:+3V3 #PWR307
 U 1 1 590237EC
 P 8800 1500
@@
 $EndComp
 $Comp
-L FT812 U301
+L usevolt:FT812 U301
 U 1 1 59252681
 P 3450 3800
@@
 $EndComp
 $Comp
-L 10K R301
+L multicomp:10K R301
 U 1 1 59C66325
 P 1400 3350
@@
 $EndComp
 $Comp
-L AL8805W5-7_LED_DRIVER U302
+L usevolt:AL8805W5-7_LED_DRIVER U302
 U 1 1 5A0D49FC
 P 7100 1400
@@
 $EndComp
 $Comp
-L 100nF C303
+L kemet:100nF C303
 U 1 1 5A0D4AC7
 P 6500 1350
@@
 	6700 1300 6700 1250
 Wire Wire Line
-	6700 1250 6250 1250
+	6700 1250 6500 1250
 Wire Wire Line
 	6800 1500 6700 1500
@@
 	6700 1500 6700 1550
 Wire Wire Line
-	6700 1550 6250 1550
-$Comp
-L GND #PWR306
+	6700 1550 6500 1550
+$Comp
+L power1:GND #PWR306
 U 1 1 5A0D4BEC
 P 6500 1650
@@
 Connection ~ 6500 1250
 Wire Wire Line
-	6500 1250 6500 750
+	6500 1250 6500 900
 Wire Wire Line
 	8250 1300 8250 1900
 Wire Wire Line
-	7400 1300 8250 1300
-$Comp
-L R_0.33OHM R302
+	7400 1300 7800 1300
+$Comp
+L usevolt:R_0.33OHM R302
 U 1 1 5A0D50A7
 P 7800 1100
@@
 Connection ~ 7800 1300
 $Comp
-L DIODE_RS07J-GS18 D301
+L usevolt:DIODE_RS07J-GS18 D301
 U 1 1 5A0D515C
 P 8450 1100
@@
 $EndComp
 Wire Wire Line
-	8450 1300 8450 1800
+	8450 1300 8450 1500
 Wire Wire Line
 	8450 900  8450 1000
 Wire Wire Line
-	6500 900  8450 900
+	6500 900  7800 900
 Connection ~ 7800 900
 Connection ~ 6500 900
 $Comp
-L IND_744045210 L301
+L usevolt:IND_744045210 L301
 U 1 1 5A0D53A4
 P 7750 1500
@@
 Connection ~ 8450 1500
 $Comp
-L VEE #PWR305
+L power1:VEE #PWR305
 U 1 1 5A0D7248
 P 6500 750
@@
 $EndComp
 $Comp
-L HEADER_MOLEX_52207-0433 J302
+L usevolt:HEADER_MOLEX_52207-0433 J302
 U 1 1 5A1297ED
 P 8250 6150
@@
 	6250 6350 8150 6350
 $Comp
-L CAP_EEE-FK1H470P C304
+L usevolt:CAP_EEE-FK1H470P C304
 U 1 1 5A12F27F
 P 6250 1450
@@
 	0    1    1    0
 $EndComp
+Wire Wire Line
+	8900 5300 8900 5800
+Wire Wire Line
+	8900 4600 8900 5300
+Wire Wire Line
+	2650 2200 2650 2300
+Wire Wire Line
+	2650 2200 2850 2200
+Wire Wire Line
+	2650 2300 2650 2400
+Wire Wire Line
+	2650 2400 2650 2500
+Wire Wire Line
+	2650 5700 2650 5800
+Wire Wire Line
+	2650 5600 2650 5700
+Wire Wire Line
+	2650 5500 2650 5600
+Wire Wire Line
+	2650 5400 2650 5500
+Wire Wire Line
+	1650 2200 2650 2200
+Wire Wire Line
+	6500 1550 6250 1550
+Wire Wire Line
+	6500 1250 6250 1250
+Wire Wire Line
+	7800 1300 8250 1300
+Wire Wire Line
+	7800 900  8450 900
+Wire Wire Line
+	6500 900  6500 750
+Wire Wire Line
+	8450 1500 8450 1800
 $EndSCHEMATC
