File: hw/tft-lcd.sch (KiCad schematic (older format))
At the start: 12 parts, among them J301 HEADER_MOLEX_54104-4031, J302 HEADER_MOLEX_52207-0433, U301 FT812, U302 AL8805W5-7_LED_DRIVER

Commit message: working rtc module for LPC1549
Parts:
- C301, C302, C303: symbol 100nF -> kemet:100nF
- C304: symbol CAP_EEE-FK1H470P -> usevolt:CAP_EEE-FK1H470P
- D301: symbol DIODE_RS07J-GS18 -> usevolt:DIODE_RS07J-GS18
- J301: symbol HEADER_MOLEX_54104-4031 -> usevolt:HEADER_MOLEX_54104-4031
- J302: symbol HEADER_MOLEX_52207-0433 -> usevolt:HEADER_MOLEX_52207-0433
- L301: symbol IND_744045210 -> usevolt:IND_744045210
- R301: symbol 10K -> multicomp:10K
- R302: symbol R_0.33OHM -> usevolt:R_0.33OHM
- U301: symbol FT812 -> usevolt:FT812
- U302: symbol AL8805W5-7_LED_DRIVER -> usevolt:AL8805W5-7_LED_DRIVER
Changed lines of the file:
@@
-EESchema Schematic File Version 2
-LIBS:display-rescue
-LIBS:kemet
-LIBS:multicomp
-LIBS:usevolt
-LIBS:wurth_elektronik_LED
-LIBS:power
+EESchema Schematic File Version 4
 LIBS:display-cache
 EELAYER 26 0
@@
 $Descr A4 11693 8268
 encoding utf-8
-Sheet 3 6
+Sheet 3 7
 Title ""
 Date ""
@@
 $EndDescr
 $Comp
-L HEADER_MOLEX_54104-4031 J301
+L usevolt:HEADER_MOLEX_54104-4031 J301
 U 1 1 58FC4B22
 P 9550 3250
@@
 YU
 $Comp
-L GND #PWR308
+L power1:GND #PWR0308
 U 1 1 58FC5C8D
 P 8900 5800
-F 0 "#PWR308" H 8900 5550 50  0001 C CNN
+F 0 "#PWR0308" H 8900 5550 50  0001 C CNN
 F 1 "GND" H 8905 5627 50  0000 C CNN
 F 2 "" H 8900 5800 50  0000 C CNN
@@
 	8800 1500 8800 2100
 $Comp
-L +3V3 #PWR303
+L power1:+3V3 #PWR0303
 U 1 1 58FC70E1
 P 2650 2100
-F 0 "#PWR303" H 2650 1950 50  0001 C CNN
+F 0 "#PWR0303" H 2650 1950 50  0001 C CNN
 F 1 "+3V3" H 2665 2273 50  0000 C CNN
 F 2 "" H 2650 2100 50  0000 C CNN
@@
 	2450 3200 2850 3200
 $Comp
-L GND #PWR304
+L power1:GND #PWR0304
 U 1 1 58FC8063
 P 2650 5800
-F 0 "#PWR304" H 2650 5550 50  0001 C CNN
+F 0 "#PWR0304" H 2650 5550 50  0001 C CNN
 F 1 "GND" H 2655 5627 50  0000 C CNN
 F 2 "" H 2650 5800 50  0000 C CNN
@@
 Connection ~ 2650 5400
 $Comp
-L 100nF C302
+L kemet:100nF C302
 U 1 1 58FC823D
 P 1650 2300
@@
 $EndComp
 $Comp
-L 100nF C301
+L kemet:100nF C301
 U 1 1 58FC82A4
 P 1300 2300
@@
 Connection ~ 1650 2200
 $Comp
-L GND #PWR301
+L power1:GND #PWR0301
 U 1 1 58FC846A
 P 1300 2550
-F 0 "#PWR301" H 1300 2300 50  0001 C CNN
+F 0 "#PWR0301" H 1300 2300 50  0001 C CNN
 F 1 "GND" H 1305 2377 50  0000 C CNN
 F 2 "" H 1300 2550 50  0000 C CNN
@@
 	1300 2550 1300 2500
 $Comp
-L +3V3 #PWR302
+L power1:+3V3 #PWR0302
 U 1 1 5900C7EB
 P 1400 3150
-F 0 "#PWR302" H 1400 3000 50  0001 C CNN
+F 0 "#PWR0302" H 1400 3000 50  0001 C CNN
 F 1 "+3V3" H 1415 3323 50  0000 C CNN
 F 2 "" H 1400 3150 50  0000 C CNN
@@
 	8450 1800 9400 1800
 $Comp
-L +3V3 #PWR307
+L power1:+3V3 #PWR0307
 U 1 1 590237EC
 P 8800 1500
-F 0 "#PWR307" H 8800 1350 50  0001 C CNN
+F 0 "#PWR0307" H 8800 1350 50  0001 C CNN
 F 1 "+3V3" H 8815 1673 50  0000 C CNN
 F 2 "" H 8800 1500 50  0000 C CNN
@@
 $EndComp
 $Comp
-L FT812 U301
+L usevolt:FT812 U301
 U 1 1 59252681
 P 3450 3800
@@
 $EndComp
 $Comp
-L 10K R301
+L multicomp:10K R301
 U 1 1 59C66325
 P 1400 3350
@@
 $EndComp
 $Comp
-L AL8805W5-7_LED_DRIVER U302
+L usevolt:AL8805W5-7_LED_DRIVER U302
 U 1 1 5A0D49FC
 P 7100 1400
@@
 $EndComp
 $Comp
-L 100nF C303
+L kemet:100nF C303
 U 1 1 5A0D4AC7
 P 6500 1350
@@
 	6700 1550 6250 1550
 $Comp
-L GND #PWR306
+L power1:GND #PWR0306
 U 1 1 5A0D4BEC
 P 6500 1650
-F 0 "#PWR306" H 6500 1400 50  0001 C CNN
+F 0 "#PWR0306" H 6500 1400 50  0001 C CNN
 F 1 "GND" H 6505 1477 50  0000 C CNN
 F 2 "" H 6500 1650 50  0000 C CNN
@@
 	7400 1300 8250 1300
 $Comp
-L R_0.33OHM R302
+L usevolt:R_0.33OHM R302
 U 1 1 5A0D50A7
 P 7800 1100
@@
 Connection ~ 7800 1300
 $Comp
-L DIODE_RS07J-GS18 D301
+L usevolt:DIODE_RS07J-GS18 D301
 U 1 1 5A0D515C
 P 8450 1100
@@
 Connection ~ 6500 900
 $Comp
-L IND_744045210 L301
+L usevolt:IND_744045210 L301
 U 1 1 5A0D53A4
 P 7750 1500
@@
 Connection ~ 8450 1500
 $Comp
-L VEE #PWR305
+L power1:VEE #PWR0305
 U 1 1 5A0D7248
 P 6500 750
-F 0 "#PWR305" H 6500 600 50  0001 C CNN
+F 0 "#PWR0305" H 6500 600 50  0001 C CNN
 F 1 "VEE" H 6517 923 50  0000 C CNN
 F 2 "" H 6500 750 50  0000 C CNN
@@
 $EndComp
 $Comp
-L HEADER_MOLEX_52207-0433 J302
+L usevolt:HEADER_MOLEX_52207-0433 J302
 U 1 1 5A1297ED
 P 8250 6150
@@
 	6250 6350 8150 6350
 $Comp
-L CAP_EEE-FK1H470P C304
+L usevolt:CAP_EEE-FK1H470P C304
 U 1 1 5A12F27F
 P 6250 1450
