File: hw/buzzer.sch (KiCad schematic (older format))
At the start: 5 parts, among them U601 OPAMP_LM358DT, X601 BUZZER_PKM13EPYH4002-B0

Commit message: kicad schematic update
Parts:
- C601: symbol 100nF -> kemet:100nF
- R601, R602: symbol 10K -> multicomp:10K
- U601: symbol OPAMP_LM358DT -> usevolt:OPAMP_LM358DT
- X601: symbol BUZZER_PKM13EPYH4002-B0 -> usevolt:BUZZER_PKM13EPYH4002-B0
Changed lines of the file:
@@
-EESchema Schematic File Version 2
-LIBS:display-rescue
-LIBS:kemet
-LIBS:multicomp
-LIBS:usevolt
-LIBS:wurth_elektronik_LED
-LIBS:power
+EESchema Schematic File Version 4
 LIBS:display-cache
 EELAYER 26 0
@@
 PWM_IN
 $Comp
-L BUZZER_PKM13EPYH4002-B0 X601
+L usevolt:BUZZER_PKM13EPYH4002-B0 X601
 U 1 1 5A1B24C9
 P 6250 3900
@@
 $EndComp
 $Comp
-L OPAMP_LM358DT U601
+L usevolt:OPAMP_LM358DT U601
 U 1 1 5A1B6095
 P 5650 3700
@@
 $EndComp
 $Comp
-L VDD #PWR603
+L power1:VDD #PWR603
 U 1 1 5A1B60F5
 P 6250 3400
@@
 	6250 3600 6050 3600
 $Comp
-L 100nF C601
+L kemet:100nF C601
 U 1 1 5A1B6111
 P 6350 3600
@@
 	6050 3700 7450 3700
 $Comp
-L GND #PWR604
+L power1:GND #PWR604
 U 1 1 5A1B615A
 P 7450 4300
@@
 	5100 3600 5350 3600
 $Comp
-L GND #PWR602
+L power1:GND #PWR602
 U 1 1 5A1B6AE9
 P 5100 4100
@@
 	5100 3800 5100 4100
 $Comp
-L 10K R601
+L multicomp:10K R601
 U 1 1 5A1B783E
 P 4400 3450
@@
 $EndComp
 $Comp
-L 10K R602
+L multicomp:10K R602
 U 1 1 5A1B78AD
 P 4400 3850
@@
 Connection ~ 5100 4050
 $Comp
-L +3V3 #PWR601
+L power1:+3V3 #PWR601
 U 1 1 5A1B792F
 P 4400 3250
