File: hw/buzzer.sch (KiCad schematic (older format))
At the start: 5 parts, among them U601 OPAMP_LM358DT, X601 BUZZER_PKM13EPYH4002-B0

Commit message: working rtc module for LPC1549
Parts:
- C601: symbol 100nF -> kemet:100nF
- R601, R602: symbol 10K -> multicomp:10K
- U601: symbol OPAMP_LM358DT -> usevolt:OPAMP_LM358DT
- X601: symbol BUZZER_PKM13EPYH4002-B0 -> usevolt:BUZZER_PKM13EPYH4002-B0
Connections:
- wire segments 15 -> 20
Changed lines of the file:
@@
-EESchema Schematic File Version 2
-LIBS:display-rescue
-LIBS:kemet
-LIBS:multicomp
-LIBS:usevolt
-LIBS:wurth_elektronik_LED
-LIBS:power
+EESchema Schematic File Version 4
 LIBS:display-cache
 EELAYER 26 0
@@
 $Descr A4 11693 8268
 encoding utf-8
-Sheet 6 6
+Sheet 6 7
 Title ""
 Date ""
@@
 PWM_IN
 $Comp
-L BUZZER_PKM13EPYH4002-B0 X601
+L usevolt:BUZZER_PKM13EPYH4002-B0 X601
 U 1 1 5A1B24C9
 P 6250 3900
@@
 $EndComp
 $Comp
-L OPAMP_LM358DT U601
+L usevolt:OPAMP_LM358DT U601
 U 1 1 5A1B6095
 P 5650 3700
@@
 $EndComp
 $Comp
-L VDD #PWR603
+L power1:VDD #PWR0603
 U 1 1 5A1B60F5
 P 6250 3400
-F 0 "#PWR603" H 6250 3250 50  0001 C CNN
+F 0 "#PWR0603" H 6250 3250 50  0001 C CNN
 F 1 "VDD" H 6267 3573 50  0000 C CNN
 F 2 "" H 6250 3400 50  0000 C CNN
@@
 	6250 3600 6050 3600
 $Comp
-L 100nF C601
+L kemet:100nF C601
 U 1 1 5A1B6111
 P 6350 3600
@@
 	6050 3700 7450 3700
 $Comp
-L GND #PWR604
+L power1:GND #PWR0604
 U 1 1 5A1B615A
 P 7450 4300
-F 0 "#PWR604" H 7450 4050 50  0001 C CNN
+F 0 "#PWR0604" H 7450 4050 50  0001 C CNN
 F 1 "GND" H 7455 4127 50  0000 C CNN
 F 2 "" H 7450 4300 50  0000 C CNN
@@
 $EndComp
 Wire Wire Line
-	7450 3600 7450 4300
+	7450 3600 7450 3700
 Connection ~ 6250 3600
 Wire Wire Line
@@
 	5100 3600 5350 3600
 $Comp
-L GND #PWR602
+L power1:GND #PWR0602
 U 1 1 5A1B6AE9
 P 5100 4100
-F 0 "#PWR602" H 5100 3850 50  0001 C CNN
+F 0 "#PWR0602" H 5100 3850 50  0001 C CNN
 F 1 "GND" H 5105 3927 50  0000 C CNN
 F 2 "" H 5100 4100 50  0000 C CNN
@@
 	5100 3800 5350 3800
 Wire Wire Line
-	5100 3800 5100 4100
+	5100 3800 5100 3900
 $Comp
-L 10K R601
+L multicomp:10K R601
 U 1 1 5A1B783E
 P 4400 3450
@@
 $EndComp
 $Comp
-L 10K R602
+L multicomp:10K R602
 U 1 1 5A1B78AD
 P 4400 3850
@@
 $EndComp
 Wire Wire Line
-	4400 3650 4400 3750
+	4400 3650 4400 3700
 Wire Wire Line
 	4400 4050 5100 4050
 Connection ~ 5100 4050
 $Comp
-L +3V3 #PWR601
+L power1:+3V3 #PWR0601
 U 1 1 5A1B792F
 P 4400 3250
-F 0 "#PWR601" H 4400 3100 50  0001 C CNN
+F 0 "#PWR0601" H 4400 3100 50  0001 C CNN
 F 1 "+3V3" H 4415 3423 50  0000 C CNN
 F 2 "" H 4400 3250 50  0000 C CNN
@@
 	5350 3700 4400 3700
 Connection ~ 4400 3700
+Wire Wire Line
+	7450 3700 7450 4100
+Wire Wire Line
+	7450 4100 7450 4300
+Wire Wire Line
+	5100 3900 5100 4050
+Wire Wire Line
+	5100 4050 5100 4100
+Wire Wire Line
+	4400 3700 4400 3750
 $EndSCHEMATC
