File: hw/flashmemory.sch (KiCad schematic (older format))
At the start: 2 parts, among them U501 WINDBOND_W25Q128JVSIQ_SOIC8_W

Commit message: kicad schematic update
Parts:
- C501: symbol 100nF -> kemet:100nF
- U501: symbol WINDBOND_W25Q128JVSIQ_SOIC8_W -> usevolt:WINDBOND_W25Q128JVSIQ_SOIC8_W
Changed lines of the file:
@@
-EESchema Schematic File Version 2
-LIBS:display-rescue
-LIBS:kemet
-LIBS:multicomp
-LIBS:usevolt
-LIBS:wurth_elektronik_LED
-LIBS:power
+EESchema Schematic File Version 4
 LIBS:display-cache
 EELAYER 26 0
@@
 $EndDescr
 $Comp
-L WINDBOND_W25Q128JVSIQ_SOIC8_W U501
+L usevolt:WINDBOND_W25Q128JVSIQ_SOIC8_W U501
 U 1 1 59C65DF2
 P 6100 2750
@@
 $EndComp
 $Comp
-L GND #PWR501
+L power1:GND #PWR501
 U 1 1 59C661EF
 P 5450 3050
@@
 	5450 2950 5600 2950
 $Comp
-L +3V3 #PWR502
+L power1:+3V3 #PWR502
 U 1 1 59C66208
 P 7600 2450
@@
 	7600 2450 7600 2700
 $Comp
-L 100nF C501
+L kemet:100nF C501
 U 1 1 59C66223
 P 7600 2800
@@
 Connection ~ 7600 2650
 $Comp
-L GND #PWR503
+L power1:GND #PWR503
 U 1 1 59C6628B
 P 7600 3100
