File: hw/lpc1549.sch (KiCad schematic (older format))
At the start: 16 parts, among them J401 ARM_JTAG_SWD_HEADER_10_PINSMD, U401 LPC1549JBD64, X401 XTAL_7A-12.000MAAJ-T, X402 XTAL_ABS25-32.768KHZ-T

Commit message: kicad schematic update
Parts:
- BT401: symbol BATTERY_HOLDER_CH7410-2032LFSMD -> usevolt:BATTERY_HOLDER_CH7410-2032LFSMD
- C401, C402, C403, C404, C405: symbol 100nF -> kemet:100nF
- C406, C407, C408, C409: symbol 18pF -> kemet:18pF
- J401: symbol ARM_JTAG_SWD_HEADER_10_PINSMD -> usevolt:ARM_JTAG_SWD_HEADER_10_PINSMD
- R405, R406: symbol 10K -> multicomp:10K
- U401: symbol LPC1549JBD64 -> usevolt:LPC1549JBD64
- X401: symbol XTAL_7A-12.000MAAJ-T -> usevolt:XTAL_7A-12.000MAAJ-T
- X402: symbol XTAL_ABS25-32.768KHZ-T -> usevolt:XTAL_ABS25-32.768KHZ-T
Connections:
- wire segments 63 -> 93
Changed lines of the file:
@@
-EESchema Schematic File Version 2
-LIBS:display-rescue
-LIBS:kemet
-LIBS:multicomp
-LIBS:usevolt
-LIBS:wurth_elektronik_LED
-LIBS:power
+EESchema Schematic File Version 4
 LIBS:display-cache
 EELAYER 26 0
@@
 $EndDescr
 $Comp
-L +3V3 #PWR401
+L power1:+3V3 #PWR401
 U 1 1 58FC1E6A
 P 4100 3150
@@
 $EndComp
 $Comp
-L 100nF C405
+L kemet:100nF C405
 U 1 1 58FC1ECE
 P 4100 3950
@@
 $EndComp
 $Comp
-L 100nF C404
+L kemet:100nF C404
 U 1 1 58FC1F13
 P 3750 3950
@@
 $EndComp
 $Comp
-L 100nF C403
+L kemet:100nF C403
 U 1 1 58FC1F6F
 P 3400 3950
@@
 $EndComp
 $Comp
-L 100nF C402
+L kemet:100nF C402
 U 1 1 58FC2016
 P 3050 3950
@@
 $EndComp
 $Comp
-L 100nF C401
+L kemet:100nF C401
 U 1 1 58FC2062
 P 2700 3950
@@
 $EndComp
 $Comp
-L GND #PWR402
+L power1:GND #PWR402
 U 1 1 58FC23D4
 P 4100 4300
@@
 LCD_CS
 $Comp
-L XTAL_7A-12.000MAAJ-T X401
+L usevolt:XTAL_7A-12.000MAAJ-T X401
 U 1 1 59022341
 P 6900 2550
@@
 $EndComp
 $Comp
-L 18pF C406
+L kemet:18pF C406
 U 1 1 590225BD
 P 7250 2350
@@
 $EndComp
 $Comp
-L 18pF C407
+L kemet:18pF C407
 U 1 1 5902262D
 P 7250 2700
@@
 $EndComp
 $Comp
-L GND #PWR405
+L power1:GND #PWR405
 U 1 1 5902271B
 P 7850 2750
@@
 $EndComp
 $Comp
-L ARM_JTAG_SWD_HEADER_10_PINSMD J401
+L usevolt:ARM_JTAG_SWD_HEADER_10_PINSMD J401
 U 1 1 59058B71
 P 9200 3700
@@
 $EndComp
 $Comp
-L +3V3 #PWR407
+L power1:+3V3 #PWR407
 U 1 1 59058BEB
 P 8900 3150
@@
 $EndComp
 $Comp
-L GND #PWR406
+L power1:GND #PWR406
 U 1 1 59058D57
 P 8750 4200
@@
 $EndComp
 $Comp
-L 10K R406
+L multicomp:10K R406
 U 1 1 59058E02
 P 8650 3500
@@
 $EndComp
 $Comp
-L 10K R405
+L multicomp:10K R405
 U 1 1 59058E98
 P 8450 3300
@@
 FLASH_CLK
 $Comp
-L 18pF C408
+L kemet:18pF C408
 U 1 1 59C7E65E
 P 7300 3100
@@
 $EndComp
 $Comp
-L 18pF C409
+L kemet:18pF C409
 U 1 1 59C7E6D2
 P 7300 3400
@@
 $EndComp
 $Comp
-L GND #PWR403
+L power1:GND #PWR403
 U 1 1 59C7ED66
 P 7550 3450
@@
 $EndComp
 $Comp
-L BATTERY_HOLDER_CH7410-2032LFSMD BT401
+L usevolt:BATTERY_HOLDER_CH7410-2032LFSMD BT401
 U 1 1 59C7EEA2
 P 7750 3400
@@
 $EndComp
 $Comp
-L GND #PWR404
+L power1:GND #PWR404
 U 1 1 59C7EFA3
 P 7750 3450
@@
 $EndComp
 $Comp
-L XTAL_ABS25-32.768KHZ-T X402
+L usevolt:XTAL_ABS25-32.768KHZ-T X402
 U 1 1 5A0A3265
 P 6700 3300
@@
 $EndComp
 $Comp
-L LPC1549JBD64 U401
+L usevolt:LPC1549JBD64 U401
 U 1 1 5A0C19C9
 P 4950 2500
@@
 $EndComp
 Wire Wire Line
-	4100 3850 4100 3150
-Wire Wire Line
-	2700 3850 4450 3850
+	4100 3850 4100 3750
+Wire Wire Line
+	2700 3850 3050 3850
 Wire Wire Line
 	4450 3750 4100 3750
@@
 Connection ~ 3050 3850
 Wire Wire Line
-	2700 4150 4450 4150
+	2700 4150 3050 4150
 Connection ~ 3050 4150
 Connection ~ 3400 4150
@@
 	4450 4250 4350 4250
 Wire Wire Line
-	4350 4150 4350 4650
+	4350 4150 4350 4250
 Connection ~ 4350 4150
 Wire Wire Line
@@
 	6250 4500 6550 4500
 Wire Wire Line
-	6250 2700 7150 2700
+	6250 2700 6900 2700
 Wire Wire Line
 	6900 2700 6900 2650
 Wire Wire Line
-	6750 2350 7150 2350
-Wire Wire Line
-	7850 2350 7850 2750
+	6750 2350 6900 2350
+Wire Wire Line
+	7850 2350 7850 2700
 Wire Wire Line
 	7850 2350 7450 2350
@@
 Connection ~ 6900 2350
 Wire Wire Line
-	8900 3150 8900 3400
-Wire Wire Line
-	8650 3400 9100 3400
+	8900 3150 8900 3200
+Wire Wire Line
+	8650 3400 8900 3400
 Wire Wire Line
 	8450 3500 9100 3500
@@
 	8450 3500 8450 3800
 Wire Wire Line
-	6450 3700 9100 3700
+	6450 3700 8650 3700
 Wire Wire Line
 	8750 4200 8750 3800
@@
 	9100 4200 9000 4200
 Wire Wire Line
-	9000 4200 9000 1100
+	9000 4200 9000 3600
 Wire Wire Line
 	9000 1100 4350 1100
@@
 	4450 2600 4150 2600
 Wire Wire Line
-	6250 3100 7200 3100
-Wire Wire Line
-	6550 3400 7200 3400
-Wire Wire Line
-	7550 3100 7550 3450
+	6250 3100 6700 3100
+Wire Wire Line
+	6550 3400 6700 3400
+Wire Wire Line
+	7550 3100 7550 3400
 Wire Wire Line
 	7550 3400 7500 3400
@@
 Text HLabel 6550 2200 2    60   Output ~ 0
 BUZZER
+Wire Wire Line
+	4100 3750 4100 3650
+Wire Wire Line
+	4100 3650 4100 3550
+Wire Wire Line
+	4100 3550 4100 3450
+Wire Wire Line
+	4100 3450 4100 3300
+Wire Wire Line
+	4100 3300 4100 3200
+Wire Wire Line
+	4100 3200 4100 3150
+Wire Wire Line
+	4100 3850 4450 3850
+Wire Wire Line
+	3750 3850 4100 3850
+Wire Wire Line
+	3400 3850 3750 3850
+Wire Wire Line
+	3050 3850 3400 3850
+Wire Wire Line
+	3050 4150 3400 4150
+Wire Wire Line
+	3400 4150 3750 4150
+Wire Wire Line
+	3750 4150 4100 4150
+Wire Wire Line
+	4100 4150 4350 4150
+Wire Wire Line
+	4350 4150 4450 4150
+Wire Wire Line
+	4350 4250 4350 4350
+Wire Wire Line
+	4350 4350 4350 4450
+Wire Wire Line
+	4350 4450 4350 4550
+Wire Wire Line
+	4350 4550 4350 4650
+Wire Wire Line
+	7850 2700 7850 2750
+Wire Wire Line
+	6900 2700 7150 2700
+Wire Wire Line
+	6900 2350 7150 2350
+Wire Wire Line
+	8650 3700 9100 3700
+Wire Wire Line
+	8900 3200 8900 3400
+Wire Wire Line
+	8900 3400 9100 3400
+Wire Wire Line
+	7550 3400 7550 3450
+Wire Wire Line
+	6700 3100 7200 3100
+Wire Wire Line
+	6700 3400 7200 3400
+Wire Wire Line
+	9100 3600 9000 3600
+Connection ~ 9000 3600
+Wire Wire Line
+	9000 3600 9000 1100
 $EndSCHEMATC
