File: hw/lpc1549.sch (KiCad schematic (older format))
At the start: 16 parts, among them J401 ARM_JTAG_SWD_HEADER_10_PINSMD, U401 LPC1549JBD64, X401 XTAL_7A-12.000MAAJ-T, X402 XTAL_ABS25-32.768KHZ-T

Commit message: working rtc module for LPC1549
Parts:
- removed BT401: BATTERY_HOLDER_CH7410-2032LFSMD, usevolt:BATTERY_HOLDER_CH7410-2032LF, symbol BATTERY_HOLDER_CH7410-2032LFSMD
- removed C408, C409: 18pF, kemet:0603, symbol 18pF
- removed X402: XTAL_ABS25-32.768KHZ-T, usevolt:XTAL_32.768KHZ-T, symbol XTAL_ABS25-32.768KHZ-T
- C401, C402, C403, C404, C405: symbol 100nF -> kemet:100nF
- C406, C407: symbol 18pF -> kemet:18pF
- J401: symbol ARM_JTAG_SWD_HEADER_10_PINSMD -> usevolt:ARM_JTAG_SWD_HEADER_10_PINSMD
- R405, R406: symbol 10K -> multicomp:10K
- U401: symbol LPC1549JBD64 -> usevolt:LPC1549JBD64
- X401: symbol XTAL_7A-12.000MAAJ-T -> usevolt:XTAL_7A-12.000MAAJ-T
Connections:
- net labels added: RTC_SCL, RTC_SDA
- wire segments 63 -> 81
Changed lines of the file:
@@
-EESchema Schematic File Version 2
-LIBS:display-rescue
-LIBS:kemet
-LIBS:multicomp
-LIBS:usevolt
-LIBS:wurth_elektronik_LED
-LIBS:power
+EESchema Schematic File Version 4
 LIBS:display-cache
 EELAYER 26 0
@@
 $Descr A4 11693 8268
 encoding utf-8
-Sheet 4 6
+Sheet 4 7
 Title ""
 Date ""
@@
 $EndDescr
 $Comp
-L +3V3 #PWR401
+L power1:+3V3 #PWR0401
 U 1 1 58FC1E6A
 P 4100 3150
-F 0 "#PWR401" H 4100 3000 50  0001 C CNN
+F 0 "#PWR0401" H 4100 3000 50  0001 C CNN
 F 1 "+3V3" H 4115 3323 50  0000 C CNN
 F 2 "" H 4100 3150 50  0000 C CNN
@@
 $EndComp
 $Comp
-L 100nF C405
+L kemet:100nF C405
 U 1 1 58FC1ECE
 P 4100 3950
@@
 $EndComp
 $Comp
-L 100nF C404
+L kemet:100nF C404
 U 1 1 58FC1F13
 P 3750 3950
@@
 $EndComp
 $Comp
-L 100nF C403
+L kemet:100nF C403
 U 1 1 58FC1F6F
 P 3400 3950
@@
 $EndComp
 $Comp
-L 100nF C402
+L kemet:100nF C402
 U 1 1 58FC2016
 P 3050 3950
@@
 $EndComp
 $Comp
-L 100nF C401
+L kemet:100nF C401
 U 1 1 58FC2062
 P 2700 3950
@@
 $EndComp
 $Comp
-L GND #PWR402
+L power1:GND #PWR0402
 U 1 1 58FC23D4
 P 4100 4300
-F 0 "#PWR402" H 4100 4050 50  0001 C CNN
+F 0 "#PWR0402" H 4100 4050 50  0001 C CNN
 F 1 "GND" H 4105 4127 50  0000 C CNN
 F 2 "" H 4100 4300 50  0000 C CNN
@@
 LCD_CS
 $Comp
-L XTAL_7A-12.000MAAJ-T X401
+L usevolt:XTAL_7A-12.000MAAJ-T X401
 U 1 1 59022341
 P 6900 2550
@@
 $EndComp
 $Comp
-L 18pF C406
+L kemet:18pF C406
 U 1 1 590225BD
 P 7250 2350
@@
 $EndComp
 $Comp
-L 18pF C407
+L kemet:18pF C407
 U 1 1 5902262D
 P 7250 2700
@@
 $EndComp
 $Comp
-L GND #PWR405
+L power1:GND #PWR0405
 U 1 1 5902271B
 P 7850 2750
-F 0 "#PWR405" H 7850 2500 50  0001 C CNN
+F 0 "#PWR0405" H 7850 2500 50  0001 C CNN
 F 1 "GND" H 7855 2577 50  0000 C CNN
 F 2 "" H 7850 2750 50  0000 C CNN
@@
 $EndComp
 $Comp
-L ARM_JTAG_SWD_HEADER_10_PINSMD J401
+L usevolt:ARM_JTAG_SWD_HEADER_10_PINSMD J401
 U 1 1 59058B71
 P 9200 3700
@@
 $EndComp
 $Comp
-L +3V3 #PWR407
+L power1:+3V3 #PWR0407
 U 1 1 59058BEB
 P 8900 3150
-F 0 "#PWR407" H 8900 3000 50  0001 C CNN
+F 0 "#PWR0407" H 8900 3000 50  0001 C CNN
 F 1 "+3V3" H 8915 3323 50  0000 C CNN
 F 2 "" H 8900 3150 50  0000 C CNN
@@
 $EndComp
 $Comp
-L GND #PWR406
+L power1:GND #PWR0406
 U 1 1 59058D57
 P 8750 4200
-F 0 "#PWR406" H 8750 3950 50  0001 C CNN
+F 0 "#PWR0406" H 8750 3950 50  0001 C CNN
 F 1 "GND" H 8755 4027 50  0000 C CNN
 F 2 "" H 8750 4200 50  0000 C CNN
@@
 $EndComp
 $Comp
-L 10K R406
+L multicomp:10K R406
 U 1 1 59058E02
 P 8650 3500
@@
 $EndComp
 $Comp
-L 10K R405
+L multicomp:10K R405
 U 1 1 59058E98
 P 8450 3300
@@
 FLASH_CLK
 $Comp
-L 18pF C408
-U 1 1 59C7E65E
-P 7300 3100
-F 0 "C408" H 7350 3299 45  0000 C CNN
-F 1 "18pF" H 7350 3215 45  0000 C CNN
-F 2 "kemet:0603" H 7330 3250 20  0001 C CNN
-F 3 "http://www.farnell.com/datasheets/2111569.pdf?_ga=1.260538573.1948984246.1460023966" H 7204 3109 60  0001 C CNN
-F 4 "1865514" H 7604 3509 60  0001 C CNN "1st Source Part Number"
-F 5 "C0603C180J2GACTU" H 7404 3309 60  0001 C CNN "Manufacturer Part Number"
-F 6 "Farnell" H 7504 3409 60  0001 C CNN "1st Source"
-F 7 "KEMET" H 7304 3209 60  0001 C CNN "Manufacturer"
-	1    7300 3100
-	1    0    0    -1
-$EndComp
-$Comp
-L 18pF C409
-U 1 1 59C7E6D2
-P 7300 3400
-F 0 "C409" H 7350 3599 45  0000 C CNN
-F 1 "18pF" H 7350 3515 45  0000 C CNN
-F 2 "kemet:0603" H 7330 3550 20  0001 C CNN
-F 3 "http://www.farnell.com/datasheets/2111569.pdf?_ga=1.260538573.1948984246.1460023966" H 7204 3409 60  0001 C CNN
-F 4 "1865514" H 7604 3809 60  0001 C CNN "1st Source Part Number"
-F 5 "C0603C180J2GACTU" H 7404 3609 60  0001 C CNN "Manufacturer Part Number"
-F 6 "Farnell" H 7504 3709 60  0001 C CNN "1st Source"
-F 7 "KEMET" H 7304 3509 60  0001 C CNN "Manufacturer"
-	1    7300 3400
-	1    0    0    -1
-$EndComp
-$Comp
-L GND #PWR403
-U 1 1 59C7ED66
-P 7550 3450
-F 0 "#PWR403" H 7550 3200 50  0001 C CNN
-F 1 "GND" H 7555 3277 50  0000 C CNN
-F 2 "" H 7550 3450 50  0000 C CNN
-F 3 "" H 7550 3450 50  0000 C CNN
-	1    7550 3450
-	1    0    0    -1
-$EndComp
-$Comp
-L BATTERY_HOLDER_CH7410-2032LFSMD BT401
-U 1 1 59C7EEA2
-P 7750 3400
-F 0 "BT401" H 7888 3600 45  0000 L CNN
-F 1 "BATTERY_HOLDER_CH7410-2032LFSMD" H 7750 3400 45  0001 L BNN
-F 2 "usevolt:BATTERY_HOLDER_CH7410-2032LF" H 7780 3550 20  0001 C CNN
-F 3 "http://www.farnell.com/datasheets/1505862.pdf?_ga=1.251637318.1948984246.1460023966" H 7800 3800 60  0001 C CNN
-F 4 "2064724" H 8000 4000 60  0001 C CNN "Manufacturer Part Number"
-F 5 "CH7410-2032LF" H 8200 4200 60  0001 C CNN "1st Source Part Number"
-F 6 "Farnell" H 8100 4100 60  0001 C CNN "1st Source"
-F 7 "MULTICOMP" H 7900 3900 60  0001 C CNN "Manufacturer"
-	1    7750 3400
-	1    0    0    -1
-$EndComp
-$Comp
-L GND #PWR404
-U 1 1 59C7EFA3
-P 7750 3450
-F 0 "#PWR404" H 7750 3200 50  0001 C CNN
-F 1 "GND" H 7755 3277 50  0000 C CNN
-F 2 "" H 7750 3450 50  0000 C CNN
-F 3 "" H 7750 3450 50  0000 C CNN
-	1    7750 3450
-	1    0    0    -1
-$EndComp
-$Comp
-L XTAL_ABS25-32.768KHZ-T X402
-U 1 1 5A0A3265
-P 6700 3300
-F 0 "X402" V 6608 3398 45  0000 L CNN
-F 1 "XTAL_ABS25-32.768KHZ-T" V 6450 2900 45  0000 L CNN
-F 2 "usevolt:XTAL_32.768KHZ-T" H 6730 3450 20  0001 C CNN
-F 3 "http://www.abracon.com/Resonators/abs25.pdf" H 6720 3320 60  0001 C CNN
-F 4 "1611824" H 7320 3920 60  0001 C CNN "2nd Source Part Number"
-F 5 "535-9166-1-ND" H 7120 3720 60  0001 C CNN "1st Source Part Number"
-F 6 "Abracon LLC" H 6820 3420 60  0001 C CNN "Manufacturer"
-F 7 "ABS25-32.768KHZ-T" H 6920 3520 60  0001 C CNN "Manufacturer Part Number"
-F 8 "Digi-Key" H 7020 3620 60  0001 C CNN "1st Source"
-F 9 "Farnell" H 7220 3820 60  0001 C CNN "2nd Source"
-	1    6700 3300
-	0    1    1    0
-$EndComp
-$Comp
-L LPC1549JBD64 U401
+L usevolt:LPC1549JBD64 U401
 U 1 1 5A0C19C9
 P 4950 2500
@@
 $EndComp
 Wire Wire Line
-	4100 3850 4100 3150
-Wire Wire Line
-	2700 3850 4450 3850
+	4100 3850 4100 3750
+Wire Wire Line
+	2700 3850 3050 3850
 Wire Wire Line
 	4450 3750 4100 3750
@@
 Connection ~ 3050 3850
 Wire Wire Line
-	2700 4150 4450 4150
+	2700 4150 3050 4150
 Connection ~ 3050 4150
 Connection ~ 3400 4150
@@
 	4450 4250 4350 4250
 Wire Wire Line
-	4350 4150 4350 4650
+	4350 4150 4350 4250
 Connection ~ 4350 4150
 Wire Wire Line
@@
 	6250 4500 6550 4500
 Wire Wire Line
-	6250 2700 7150 2700
+	6250 2700 6900 2700
 Wire Wire Line
 	6900 2700 6900 2650
 Wire Wire Line
-	6750 2350 7150 2350
-Wire Wire Line
-	7850 2350 7850 2750
+	6750 2350 6900 2350
+Wire Wire Line
+	7850 2350 7850 2700
 Wire Wire Line
 	7850 2350 7450 2350
@@
 Connection ~ 6900 2350
 Wire Wire Line
-	8900 3150 8900 3400
-Wire Wire Line
-	8650 3400 9100 3400
+	8900 3150 8900 3200
+Wire Wire Line
+	8650 3400 8900 3400
 Wire Wire Line
 	8450 3500 9100 3500
@@
 	8450 3500 8450 3800
 Wire Wire Line
-	6450 3700 9100 3700
+	6450 3700 8650 3700
 Wire Wire Line
 	8750 4200 8750 3800
@@
 	4450 2600 4150 2600
 Wire Wire Line
-	6250 3100 7200 3100
-Wire Wire Line
-	6550 3400 7200 3400
-Wire Wire Line
-	7550 3100 7550 3450
-Wire Wire Line
-	7550 3400 7500 3400
-Wire Wire Line
-	7550 3100 7500 3100
-Connection ~ 7550 3400
-Wire Wire Line
-	7750 3000 6250 3000
-Wire Wire Line
-	7750 3450 7750 3400
-Connection ~ 6700 3100
-Connection ~ 6700 3400
-Wire Wire Line
-	6250 3200 6550 3200
-Wire Wire Line
-	6550 3200 6550 3400
-Wire Wire Line
 	6250 3400 6450 3400
 Wire Wire Line
@@
 Text HLabel 6550 2200 2    60   Output ~ 0
 BUZZER
+Wire Wire Line
+	4100 3750 4100 3650
+Wire Wire Line
+	4100 3650 4100 3550
+Wire Wire Line
+	4100 3550 4100 3450
+Wire Wire Line
+	4100 3450 4100 3300
+Wire Wire Line
+	4100 3300 4100 3200
+Wire Wire Line
+	4100 3200 4100 3150
+Wire Wire Line
+	4100 3850 4450 3850
+Wire Wire Line
+	3750 3850 4100 3850
+Wire Wire Line
+	3400 3850 3750 3850
+Wire Wire Line
+	3050 3850 3400 3850
+Wire Wire Line
+	3050 4150 3400 4150
+Wire Wire Line
+	3400 4150 3750 4150
+Wire Wire Line
+	3750 4150 4100 4150
+Wire Wire Line
+	4100 4150 4350 4150
+Wire Wire Line
+	4350 4150 4450 4150
+Wire Wire Line
+	4350 4250 4350 4350
+Wire Wire Line
+	4350 4350 4350 4450
+Wire Wire Line
+	4350 4450 4350 4550
+Wire Wire Line
+	4350 4550 4350 4650
+Wire Wire Line
+	7850 2700 7850 2750
+Wire Wire Line
+	6900 2700 7150 2700
+Wire Wire Line
+	6900 2350 7150 2350
+Wire Wire Line
+	8650 3700 9100 3700
+Wire Wire Line
+	8900 3200 8900 3400
+Wire Wire Line
+	8900 3400 9100 3400
+Wire Wire Line
+	6250 4100 6550 4100
+Wire Wire Line
+	6250 4200 6550 4200
+Text HLabel 6550 4200 2    60   BiDi ~ 0
+RTC_SDA
+Text HLabel 6550 4100 2    60   BiDi ~ 0
+RTC_SCL
 $EndSCHEMATC
