File: hw/display.sch (KiCad schematic (older format))
At the start: 3 parts, among them J101 AMPSEAL_8_POS_VERT_BLACK_SEAL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, U101 MCP2551_SOIC8

Commit message: working rtc module for LPC1549
Parts:
- C101: symbol 100nF -> kemet:100nF
- J101: symbol AMPSEAL_8_POS_VERT_BLACK_SEALED_1-776276-1 -> usevolt:AMPSEAL_8_POS_VERT_BLACK_SEALED_1-776276-1
- U101: symbol MCP2551_SOIC8 -> usevolt:MCP2551_SOIC8
Connections:
- wire segments 48 -> 51
Changed lines of the file:
@@
-EESchema Schematic File Version 2
-LIBS:display-rescue
-LIBS:kemet
-LIBS:multicomp
-LIBS:usevolt
-LIBS:wurth_elektronik_LED
-LIBS:power
+EESchema Schematic File Version 4
 LIBS:display-cache
 EELAYER 26 0
@@
 $Descr A4 11693 8268
 encoding utf-8
-Sheet 1 6
+Sheet 1 7
 Title "UV0A_hds"
 Date "2017-04-22"
@@
 $EndSheet
 $Comp
-L GND #PWR101
+L power1:GND #PWR0101
 U 1 1 58FBFAD2
 P 1900 2150
-F 0 "#PWR101" H 1900 1900 50  0001 C CNN
+F 0 "#PWR0101" H 1900 1900 50  0001 C CNN
 F 1 "GND" H 1905 1977 50  0000 C CNN
 F 2 "" H 1900 2150 50  0000 C CNN
@@
 $EndComp
 $Comp
-L 100nF C101
+L kemet:100nF C101
 U 1 1 58FBFBBE
 P 3050 2600
@@
 $EndComp
 $Comp
-L GND #PWR103
+L power1:GND #PWR0103
 U 1 1 58FC1671
 P 3050 2850
-F 0 "#PWR103" H 3050 2600 50  0001 C CNN
+F 0 "#PWR0103" H 3050 2600 50  0001 C CNN
 F 1 "GND" H 3055 2677 50  0000 C CNN
 F 2 "" H 3050 2850 50  0000 C CNN
@@
 $EndComp
 $Comp
-L +5V #PWR102
+L power1:+5V #PWR0102
 U 1 1 58FC16F6
 P 3050 2400
-F 0 "#PWR102" H 3050 2250 50  0001 C CNN
+F 0 "#PWR0102" H 3050 2250 50  0001 C CNN
 F 1 "+5V" H 3065 2573 50  0000 C CNN
 F 2 "" H 3050 2400 50  0000 C CNN
@@
 $EndComp
 $Comp
-L +5V #PWR106
+L power1:+5V #PWR0106
 U 1 1 58FC1761
 P 4000 1400
-F 0 "#PWR106" H 4000 1250 50  0001 C CNN
+F 0 "#PWR0106" H 4000 1250 50  0001 C CNN
 F 1 "+5V" H 4015 1573 50  0000 C CNN
 F 2 "" H 4000 1400 50  0000 C CNN
@@
 $EndComp
 $Comp
-L +3V3 #PWR107
+L power1:+3V3 #PWR0107
 U 1 1 58FC17CE
 P 4150 1600
-F 0 "#PWR107" H 4150 1450 50  0001 C CNN
+F 0 "#PWR0107" H 4150 1450 50  0001 C CNN
 F 1 "+3V3" H 4165 1773 50  0000 C CNN
 F 2 "" H 4150 1600 50  0000 C CNN
@@
 F12 "FLASH_CLK" O R 6400 3100 60
 F13 "BUZZER" O R 6400 4000 60
-$EndSheet
-Wire Wire Line
-	1900 1600 1900 2150
+F14 "RTC_SDA" B L 4200 3850 60
+F15 "RTC_SCL" B L 4200 3950 60
+$EndSheet
+Wire Wire Line
+	1900 1600 1900 2050
 Wire Wire Line
 	1900 1600 2400 1600
@@
 	6900 2900 6400 2900
 $Comp
-L MCP2551_SOIC8 U101
+L usevolt:MCP2551_SOIC8 U101
 U 1 1 5A0A3632
 P 2650 2600
@@
 $EndComp
 $Comp
-L AMPSEAL_8_POS_VERT_BLACK_SEALED_1-776276-1 J101
+L usevolt:AMPSEAL_8_POS_VERT_BLACK_SEALED_1-776276-1 J101
 U 1 1 5A0C087E
 P 950 1900
@@
 $EndComp
 $Comp
-L AMPSEAL_8_POS_VERT_BLACK_SEALED_1-776276-1 J101
+L usevolt:AMPSEAL_8_POS_VERT_BLACK_SEALED_1-776276-1 J101
 U 2 1 5A0C0C0A
 P 950 2050
@@
 $EndComp
 $Comp
-L AMPSEAL_8_POS_VERT_BLACK_SEALED_1-776276-1 J101
+L usevolt:AMPSEAL_8_POS_VERT_BLACK_SEALED_1-776276-1 J101
 U 3 1 5A0C0D57
 P 950 2200
@@
 $EndComp
 $Comp
-L AMPSEAL_8_POS_VERT_BLACK_SEALED_1-776276-1 J101
+L usevolt:AMPSEAL_8_POS_VERT_BLACK_SEALED_1-776276-1 J101
 U 4 1 5A0C0EAB
 P 950 2350
@@
 $EndComp
 $Comp
-L AMPSEAL_8_POS_VERT_BLACK_SEALED_1-776276-1 J101
+L usevolt:AMPSEAL_8_POS_VERT_BLACK_SEALED_1-776276-1 J101
 U 5 1 5A0C1002
 P 950 2500
@@
 $EndComp
 $Comp
-L AMPSEAL_8_POS_VERT_BLACK_SEALED_1-776276-1 J101
+L usevolt:AMPSEAL_8_POS_VERT_BLACK_SEALED_1-776276-1 J101
 U 6 1 5A0C115C
 P 950 2650
@@
 $EndComp
 $Comp
-L AMPSEAL_8_POS_VERT_BLACK_SEALED_1-776276-1 J101
+L usevolt:AMPSEAL_8_POS_VERT_BLACK_SEALED_1-776276-1 J101
 U 7 1 5A0C12B9
 P 950 2800
@@
 $EndComp
 $Comp
-L AMPSEAL_8_POS_VERT_BLACK_SEALED_1-776276-1 J101
+L usevolt:AMPSEAL_8_POS_VERT_BLACK_SEALED_1-776276-1 J101
 U 8 1 5A0C167F
 P 950 2950
@@
 $EndComp
 $Comp
-L VDD #PWR105
+L power1:VDD #PWR0105
 U 1 1 5A0D6E53
 P 3900 1200
-F 0 "#PWR105" H 3900 1050 50  0001 C CNN
+F 0 "#PWR0105" H 3900 1050 50  0001 C CNN
 F 1 "VDD" H 3917 1373 50  0000 C CNN
 F 2 "" H 3900 1200 50  0000 C CNN
@@
 	3900 1300 3600 1300
 $Comp
-L VEE #PWR104
+L power1:VEE #PWR0104
 U 1 1 5A0D70BB
 P 3750 1000
-F 0 "#PWR104" H 3750 850 50  0001 C CNN
+F 0 "#PWR0104" H 3750 850 50  0001 C CNN
 F 1 "VEE" H 3767 1173 50  0000 C CNN
 F 2 "" H 3750 1000 50  0000 C CNN
@@
 	1050 2050 1900 2050
 Connection ~ 1900 2050
+Wire Wire Line
+	1900 2050 1900 2150
+$Sheet
+S 2650 3750 1050 300
+U 5B04E397
+F0 "Sheet5B04E396" 60
+F1 "rtc.sch" 60
+F2 "SDA" B R 3700 3850 60
+F3 "SCL" B R 3700 3950 60
+$EndSheet
+Wire Wire Line
+	4200 3850 3700 3850
+Wire Wire Line
+	3700 3950 4200 3950
 $EndSCHEMATC

Commit message: displa pcb reverted back to 1.6.0 revision and imporved to 1.7.0
Parts:
- removed J101: AMPSEAL_8_POS_VERT_BLACK_SEALED_1-776276-1, usevolt:AMPSEAL_8_POS_776275-1, symbol usevolt:AMPSEAL_8_POS_VERT_BLACK_SEALED_1-776276-1
- removed U101: MCP2551_SOIC8, usevolt:SOIC8, symbol usevolt:MCP2551_SOIC8
- added BT1: BATTERY_HOLDER_CH7410-2032LFSMD, usevolt:usevolt-BATTERY_HOLDER_CH7410-2032LF, symbol usevolt:BATTERY_HOLDER_CH7410-2032LFSMD
- added C1, C2, C3, C32, C4, C5, C6, C7: 100nF, kemet:Kemet-CAPC1608X85N, symbol kemet:100nF
- added C22, C29: 12pF, kemet:Kemet-CAPC1608X85N, symbol kemet:12pF
- added D101: DIODE_RS07J-GS18, usevolt:DO219AB, symbol usevolt:DIODE_RS07J-GS18
- added J1: AMPSEAL_8_POS_776275-1, usevolt:AMPSEAL_8_POS_776275-1, symbol display-rescue:AMPSEAL_8_POS_776275-1
- added J101: HEADER_MOLEX_54104-4031, usevolt:HEADER_MOLEX_54104-4031, symbol usevolt:HEADER_MOLEX_54104-4031
- added J4: HEADER_MOLEX_52207-0433, usevolt:HEADER_MOLEX_52207-0433, symbol usevolt:HEADER_MOLEX_52207-0433
- added L101: INDUCTOR_SDR1005-101KL, usevolt:INDUCTOR_BOURNS_10X13X5MM, symbol usevolt:INDUCTOR_SDR1005-101KL
- added R101: R_0.33OHM, usevolt:0603, symbol usevolt:R_0.33OHM
- added U1: MCP2551_SOIC8, usevolt:SOIC8, symbol display-rescue:MCP2551_SOIC8-RESCUE-display
- added U102: AL8805W5-7_LED_DRIVER, usevolt:SOT-25, symbol usevolt:AL8805W5-7_LED_DRIVER
- added U2: ALLIANCE_AS4C4M16SA_TSOP_II, usevolt:TSOP_II_54_PIN, symbol usevolt:ALLIANCE_AS4C4M16SA_TSOP_II
- added X101: XTAL_ABS25-32.768KHZ-T, usevolt:XTAL_32.768KHZ-T, symbol usevolt:XTAL_ABS25-32.768KHZ-T
Connections:
- net labels added: A0, A1, A10, A11, A2, A3, A4, A5, A6, A7, A8, A9, B0, B1, B2, B3, B4, BA0, BA1, BACKLIGHT, BCKL+, BCKL-, DCLK, DE, DQ0, DQ1, DQ10, DQ11, DQ12, DQ13, DQ14, DQ15, DQ2, DQ3, DQ4, DQ5, DQ6, DQ7, DQ8, DQ9, G0, G1, G2, G3, G4, G5, HSYNC, PWR, R0, R1, R2, R3, R4, VSYNC
- net labels removed: VDD, VEE
- wire segments 51 -> 282
- no-connect marks 0 -> 3
