File: hw/lpc1785_sheet.sch (KiCad schematic (older format))
At the start: 23 parts, among them J2 ARM_JTAG_SWD_HEADER_10_PINSMD, U4 LPC1785FBD208_551QFP50, X1 XTAL_7A-20.000MAAJ-T

Commit message: displa pcb reverted back to 1.6.0 revision and imporved to 1.7.0
Parts:
- removed R?: 1K, multicomp:0603, symbol 1K
- added R301: 10K, multicomp:0603, symbol multicomp:10K
- C14, C15, C16, C17, C18, C19, C20, C21, C23, C24, C25, C26, C27, C28: symbol 100nF -> kemet:100nF
- C30, C31: symbol 18pF -> kemet:18pF
- J2: symbol ARM_JTAG_SWD_HEADER_10_PINSMD -> usevolt:ARM_JTAG_SWD_HEADER_10_PINSMD
- R5, R6, R7: symbol 10K -> multicomp:10K
- U4: symbol LPC1785FBD208_551QFP50-RESCUE-display -> display-rescue:LPC1785FBD208_551QFP50-RESCUE-display
- X1: symbol XTAL_7A-20.000MAAJ-T -> usevolt:XTAL_7A-20.000MAAJ-T
Connections:
- net GND: now also R301.1 (R1)
- net LCD_BACKLIGHT: now also R301.2 (R2)
Changed lines of the file:
@@
-EESchema Schematic File Version 2
-LIBS:display-rescue
-LIBS:kemet
-LIBS:multicomp
-LIBS:usevolt
-LIBS:wurth_elektronik_LED
-LIBS:power
-LIBS:elt21300_kicad
+EESchema Schematic File Version 4
 LIBS:display-cache
 EELAYER 26 0
@@
 $EndDescr
 $Comp
-L LPC1785FBD208_551QFP50-RESCUE-display U4
+L display-rescue:LPC1785FBD208_551QFP50-RESCUE-display U4
 U 1 1 57B485E7
 P 6700 5400
@@
 $EndComp
 $Comp
-L LPC1785FBD208_551QFP50-RESCUE-display U4
+L display-rescue:LPC1785FBD208_551QFP50-RESCUE-display U4
 U 2 1 57B48643
 P 13000 5050
@@
 $EndComp
 $Comp
-L LPC1785FBD208_551QFP50-RESCUE-display U4
+L display-rescue:LPC1785FBD208_551QFP50-RESCUE-display U4
 U 3 1 57B486B3
 P 5950 10500
@@
 $EndComp
 $Comp
-L LPC1785FBD208_551QFP50-RESCUE-display U4
+L display-rescue:LPC1785FBD208_551QFP50-RESCUE-display U4
 U 4 1 57B4870D
 P 12800 10600
@@
 $EndComp
 $Comp
-L 100nF C21
+L kemet:100nF C21
 U 1 1 57B554CA
 P 5150 4100
@@
 $EndComp
 $Comp
-L 100nF C20
+L kemet:100nF C20
 U 1 1 57B5550F
 P 5000 4100
@@
 $EndComp
 $Comp
-L 100nF C18
+L kemet:100nF C18
 U 1 1 57B5555D
 P 4850 4100
@@
 $EndComp
 $Comp
-L 100nF C16
+L kemet:100nF C16
 U 1 1 57B555AE
 P 4700 4100
@@
 Connection ~ 5150 4300
 $Comp
-L GND #PWR306
+L display-rescue:GND #PWR0306
 U 1 1 57B559C7
 P 4700 4400
-F 0 "#PWR306" H 4700 4150 50  0001 C CNN
+F 0 "#PWR0306" H 4700 4150 50  0001 C CNN
 F 1 "GND" H 4705 4227 50  0000 C CNN
 F 2 "" H 4700 4400 50  0000 C CNN
@@
 	4700 4400 4700 4300
 $Comp
-L GND #PWR308
+L display-rescue:GND #PWR0308
 U 1 1 57B55D95
 P 5400 5550
-F 0 "#PWR308" H 5400 5300 50  0001 C CNN
+F 0 "#PWR0308" H 5400 5300 50  0001 C CNN
 F 1 "GND" H 5405 5377 50  0000 C CNN
 F 2 "" H 5400 5550 50  0000 C CNN
@@
 Connection ~ 5400 5500
 $Comp
-L ARM_JTAG_SWD_HEADER_10_PINSMD J2
+L usevolt:ARM_JTAG_SWD_HEADER_10_PINSMD J2
 U 1 1 57B56492
 P 3800 4950
@@
 $EndComp
 $Comp
-L 10K R5
+L multicomp:10K R5
 U 1 1 57B56555
 P 4150 4450
@@
 $EndComp
 $Comp
-L 10K R6
+L multicomp:10K R6
 U 1 1 57B565D1
 P 4250 4450
@@
 $EndComp
 $Comp
-L 10K R7
+L multicomp:10K R7
 U 1 1 57B56630
 P 4350 4450
@@
 $EndComp
 $Comp
-L +3V3 #PWR305
+L display-rescue:+3V3 #PWR305
 U 1 1 57B596F9
 P 4700 3900
-F 0 "#PWR305" H 4700 3750 50  0001 C CNN
+AR Path="/57B596F9" Ref="#PWR305"  Part="1"
+AR Path="/57B4853E/57B596F9" Ref="#PWR0305"  Part="1"
+F 0 "#PWR0305" H 4700 3750 50  0001 C CNN
 F 1 "+3V3" H 4715 4073 50  0000 C CNN
 F 2 "" H 4700 3900 50  0000 C CNN
@@
 $EndComp
 $Comp
-L +3V3 #PWR302
+L display-rescue:+3V3 #PWR302
 U 1 1 57B59727
 P 4150 4250
-F 0 "#PWR302" H 4150 4100 50  0001 C CNN
+AR Path="/57B59727" Ref="#PWR302"  Part="1"
+AR Path="/57B4853E/57B59727" Ref="#PWR0302"  Part="1"
+F 0 "#PWR0302" H 4150 4100 50  0001 C CNN
 F 1 "+3V3" H 4165 4423 50  0000 C CNN
 F 2 "" H 4150 4250 50  0000 C CNN
@@
 Connection ~ 4250 4950
 $Comp
-L GND #PWR301
+L display-rescue:GND #PWR0301
 U 1 1 57B59EBE
 P 4050 5550
-F 0 "#PWR301" H 4050 5300 50  0001 C CNN
+F 0 "#PWR0301" H 4050 5300 50  0001 C CNN
 F 1 "GND" H 4055 5377 50  0000 C CNN
 F 2 "" H 4050 5550 50  0000 C CNN
@@
 	10850 3850 11300 3850
 $Comp
-L 100nF C24
+L kemet:100nF C24
 U 1 1 57B60D49
 P 10850 3950
@@
 $EndComp
 $Comp
-L 100nF C26
+L kemet:100nF C26
 U 1 1 57B60CDA
 P 11000 3950
@@
 $EndComp
 $Comp
-L 100nF C28
+L kemet:100nF C28
 U 1 1 57B60C56
 P 11150 3950
@@
 	16500 6650 16400 6650
 $Comp
-L 100nF C19
+L kemet:100nF C19
 U 1 1 57B6835D
 P 4850 9500
@@
 $EndComp
 $Comp
-L 100nF C17
+L kemet:100nF C17
 U 1 1 57B683E5
 P 4700 9500
@@
 $EndComp
 $Comp
-L 100nF C15
+L kemet:100nF C15
 U 1 1 57B68462
 P 4550 9500
@@
 $EndComp
 $Comp
-L 100nF C14
+L kemet:100nF C14
 U 1 1 57B68547
 P 4400 9500
@@
 	9050 11500 9150 11500
 $Comp
-L 100nF C27
+L kemet:100nF C27
 U 1 1 57B6E6F9
 P 11050 9000
@@
 $EndComp
 $Comp
-L 100nF C25
+L kemet:100nF C25
 U 1 1 57B6E794
 P 10900 9000
@@
 $EndComp
 $Comp
-L 100nF C23
+L kemet:100nF C23
 U 1 1 57B6E8AC
 P 10750 9000
@@
 Connection ~ 11700 9000
 $Comp
-L GND #PWR310
+L display-rescue:GND #PWR0310
 U 1 1 57B6EDB0
 P 10750 9250
-F 0 "#PWR310" H 10750 9000 50  0001 C CNN
+F 0 "#PWR0310" H 10750 9000 50  0001 C CNN
 F 1 "GND" H 10755 9077 50  0000 C CNN
 F 2 "" H 10750 9250 50  0000 C CNN
@@
 Connection ~ 10900 9200
 $Comp
-L XTAL_7A-20.000MAAJ-T X1
+L usevolt:XTAL_7A-20.000MAAJ-T X1
 U 1 1 57B6F0AD
 P 11600 9400
@@
 	11750 9200 11500 9200
 $Comp
-L 18pF C30
+L kemet:18pF C30
 U 1 1 57B6F4C3
 P 11300 9200
@@
 $EndComp
 $Comp
-L 18pF C31
+L kemet:18pF C31
 U 1 1 57B6F533
 P 11300 9500
@@
 	11200 9200 11200 9500
 $Comp
-L GND #PWR313
+L display-rescue:GND #PWR0313
 U 1 1 57B6F87A
 P 11100 9400
-F 0 "#PWR313" H 11100 9150 50  0001 C CNN
+F 0 "#PWR0313" H 11100 9150 50  0001 C CNN
 F 1 "GND" H 11105 9227 50  0000 C CNN
 F 2 "" H 11100 9400 50  0000 C CNN
@@
 Connection ~ 11700 9700
 $Comp
-L GND #PWR314
+L display-rescue:GND #PWR0314
 U 1 1 57B7073F
 P 11700 9850
-F 0 "#PWR314" H 11700 9600 50  0001 C CNN
+F 0 "#PWR0314" H 11700 9600 50  0001 C CNN
 F 1 "GND" H 11705 9677 50  0000 C CNN
 F 2 "" H 11700 9850 50  0000 C CNN
@@
 $Bitmap
 Pos 22650 15250
-Scale 1,000000
+Scale 1.000000
 Data
 89 50 4E 47 0D 0A 1A 0A 00 00 00 0D 49 48 44 52 00 00 00 7B 00 00 00 49 08 02 00 00 00 92 17 CE
@@
 SPI_RESET
 $Comp
-L +3V3 #PWR309
+L display-rescue:+3V3 #PWR309
 U 1 1 57BCA081
 P 10750 8800
-F 0 "#PWR309" H 10750 8650 50  0001 C CNN
+AR Path="/57BCA081" Ref="#PWR309"  Part="1"
+AR Path="/57B4853E/57BCA081" Ref="#PWR0309"  Part="1"
+F 0 "#PWR0309" H 10750 8650 50  0001 C CNN
 F 1 "+3V3" H 10765 8973 50  0000 C CNN
 F 2 "" H 10750 8800 50  0000 C CNN
@@
 	10750 8800 10750 8900
 $Comp
-L +3V3 #PWR303
+L display-rescue:+3V3 #PWR303
 U 1 1 57BCA489
 P 4400 9250
-F 0 "#PWR303" H 4400 9100 50  0001 C CNN
+AR Path="/57BCA489" Ref="#PWR303"  Part="1"
+AR Path="/57B4853E/57BCA489" Ref="#PWR0303"  Part="1"
+F 0 "#PWR0303" H 4400 9100 50  0001 C CNN
 F 1 "+3V3" H 4415 9423 50  0000 C CNN
 F 2 "" H 4400 9250 50  0000 C CNN
@@
 	4400 9250 4400 9400
 $Comp
-L +3V3 #PWR311
+L display-rescue:+3V3 #PWR311
 U 1 1 57BCB2A0
 P 10850 3700
-F 0 "#PWR311" H 10850 3550 50  0001 C CNN
+AR Path="/57BCB2A0" Ref="#PWR311"  Part="1"
+AR Path="/57B4853E/57BCB2A0" Ref="#PWR0311"  Part="1"
+F 0 "#PWR0311" H 10850 3550 50  0001 C CNN
 F 1 "+3V3" H 10865 3873 50  0000 C CNN
 F 2 "" H 10850 3700 50  0000 C CNN
@@
 	10850 3700 10850 3850
 $Comp
-L GND #PWR312
+L display-rescue:GND #PWR0312
 U 1 1 57BCB9E7
 P 10850 4300
-F 0 "#PWR312" H 10850 4050 50  0001 C CNN
+F 0 "#PWR0312" H 10850 4050 50  0001 C CNN
 F 1 "GND" H 10855 4127 50  0000 C CNN
 F 2 "" H 10850 4300 50  0000 C CNN
@@
 	10850 4300 10850 4150
 $Comp
-L GND #PWR304
+L display-rescue:GND #PWR0304
 U 1 1 57BCC515
 P 4400 9850
-F 0 "#PWR304" H 4400 9600 50  0001 C CNN
+F 0 "#PWR0304" H 4400 9600 50  0001 C CNN
 F 1 "GND" H 4405 9677 50  0000 C CNN
 F 2 "" H 4400 9850 50  0000 C CNN
@@
 Connection ~ 5350 7300
 $Comp
-L GND #PWR307
+L display-rescue:GND #PWR0307
 U 1 1 59507EAE
 P 5350 7800
-F 0 "#PWR307" H 5350 7550 50  0001 C CNN
+F 0 "#PWR0307" H 5350 7550 50  0001 C CNN
 F 1 "GND" H 5355 7627 50  0000 C CNN
 F 2 "" H 5350 7800 50  0000 C CNN
@@
 	5350 7800 5350 7700
 $Comp
-L 1K R?
-U 1 1 59515664
+L multicomp:10K R301
+U 1 1 595084C8
 P 5350 7500
-F 0 "R?" V 5358 7558 45  0000 L CNN
-F 1 "1K" V 5442 7558 45  0000 L CNN
+F 0 "R301" V 5358 7558 45  0000 L CNN
+F 1 "10K" V 5442 7558 45  0000 L CNN
 F 2 "multicomp:0603" H 5380 7650 20  0001 C CNN
-F 3 "" H 5319 7539 60  0001 C CNN
-F 4 "9330380" H 5719 7939 60  0001 C CNN "1st Source Part Number"
+F 3 "http://www.farnell.com/datasheets/1788326.pdf?_ga=1.214208087.1948984246.1460023966" H 5319 7539 60  0001 C CNN
+F 4 "9330399" H 5719 7939 60  0001 C CNN "1st Source Part Number"
 F 5 "Farnell" H 5619 7839 60  0001 C CNN "1st Source"
-F 6 "MC0063W060311K" H 5519 7739 60  0001 C CNN "Manufacturer Part Number"
+F 6 "MC0063W0603110K" H 5519 7739 60  0001 C CNN "Manufacturer Part Number"
 F 7 "MULTICOMP" H 5419 7639 60  0001 C CNN "Manufacturer"
 	1    5350 7500
